Commit message: camera integrated, some changes to launch sequence and updated urdf

File: patrol_description/urdf/patrol.urdf.xacro (robot description, xacro)
@@ -28,7 +28,7 @@
   <link name="base_link">
     <visual>
-      <origin xyz="0 0 0" rpy="0 0 ${-pi/2}" />
+      <origin xyz="0 0 0" rpy="${pi/2} 0 0" />
       <geometry>
-        <mesh filename="package://patrol_description/meshes/base_link.STL" />
+        <mesh filename="package://patrol_description/meshes/ANCS-000.STL" />
       </geometry>
       <material name="white"/>
@@ -60,7 +60,7 @@
     <child link="inertial_link" />
   </joint>
-  <!-- Adjust origin to TiM sensor mount-->
+  <!-- 0.165 -->
   <joint name="laser_tim_mount_joint" type="fixed">
-    <origin xyz="0.75 0 0.2" rpy="0 0 0" />
+    <origin xyz="0.69791 0 0.162" rpy="0 0.349 0" />
     <parent link="base_link" />
     <child link="laser_tim_mount_link" />
@@ -68,5 +68,5 @@
   <!-- Adjust origin to LMS sensor mount-->
   <joint name="laser_lms_mount_joint" type="fixed">
-    <origin xyz="0.55 0 0.5" rpy="0 0 0" />
+    <origin xyz="0.5288 0 0.47026" rpy="0 0 0" />
     <parent link="base_link" />
     <child link="laser_lms_mount_link" />
@@ -111,11 +111,11 @@
   <xacro:if value="${realsense_enabled}">
     <xacro:sensor_d435i parent="base_link" name="cam0" use_nominal_extrinsics="$(arg use_nominal_extrinsics)">
-      <origin xyz="2 0 0" rpy="0 0 0"/>
+      <origin xyz="-0.12213 -0.00228 0.69821" rpy="0 0 0"/>
     </xacro:sensor_d435i>
     <xacro:sensor_d435i parent="base_link" name="cam1" use_nominal_extrinsics="$(arg use_nominal_extrinsics)">
-      <origin xyz="2 0.2 0" rpy="0 0 ${pi/2}"/>
+      <origin xyz="-0.2489 0.1793 0.69821" rpy="0 0 ${pi/2}"/>
     </xacro:sensor_d435i>
     <xacro:sensor_d435i parent="base_link" name="cam2" use_nominal_extrinsics="$(arg use_nominal_extrinsics)">
-      <origin xyz="2 -0.2 0" rpy="0 0 ${-pi/2}"/>
+      <origin xyz="-0.2489 -0.17925 0.69821" rpy="0 0 ${-pi/2}"/>
     </xacro:sensor_d435i>
   </xacro:if>

Commit message: changes to URDF and launch sequence

File: patrol_description/urdf/patrol.urdf.xacro (robot description, xacro)
@@ -30,5 +30,5 @@
       <origin xyz="0 0 0" rpy="${pi/2} 0 0" />
       <geometry>
-        <mesh filename="package://patrol_description/meshes/ANCS-000.STL" />
+        <mesh filename="package://patrol_description/meshes/ANCS-000-R1.STL" />
       </geometry>
       <material name="white"/>
@@ -59,4 +59,28 @@
     <parent link="base_link" />
     <child link="inertial_link" />
+  </joint>
+  <link name="imu_link">
+    <inertial>
+      <origin xyz="0 0 0" rpy="0 0 0"/>
+      <mass value="0.1"/>
+      <inertia ixx="0.01" ixy="0" ixz="0" iyy="0.01" iyz="0" izz="0.01"/>
+    </inertial>
+  </link>
+  <joint name="imu_joint" type="fixed">
+    <parent link="base_link"/>
+    <child link="imu_link"/>
+    <origin xyz="0.193 0.0868 0.27458" rpy="0 0 0"/>
+  </joint>
+  <link name="gps">
+    <inertial>
+      <origin xyz="0 0 0" rpy="0 0 0"/>
+      <mass value="0.1"/>
+      <inertia ixx="0.01" ixy="0" ixz="0" iyy="0.01" iyz="0" izz="0.01"/>
+    </inertial>
+  </link>
+  <joint name="gps_joint" type="fixed">
+    <parent link="base_link"/>
+    <child link="gps"/>
+    <origin xyz="-0.2489 -0.11358 0.86478" rpy="0 0 0"/>
   </joint>
   <!-- 0.165 -->
@@ -111,5 +135,5 @@
   <xacro:if value="${realsense_enabled}">
     <xacro:sensor_d435i parent="base_link" name="cam0" use_nominal_extrinsics="$(arg use_nominal_extrinsics)">
-      <origin xyz="-0.12213 -0.00228 0.69821" rpy="0 0 0"/>
+      <origin xyz="-0.11913 -0.00228 0.78821" rpy="0 0 0"/>
     </xacro:sensor_d435i>
     <xacro:sensor_d435i parent="base_link" name="cam1" use_nominal_extrinsics="$(arg use_nominal_extrinsics)">

Commit message: launch changes

File: patrol_description/urdf/patrol.urdf.xacro (robot description, xacro)
@@ -14,5 +14,5 @@
   <!-- Xacro arguments for realsense d435i camera -->
   <xacro:property name="realsense_enabled" value="$(optenv REALSENSE_ENABLE false)"/>
-  <xacro:arg name="use_nominal_extrinsics" default="false"/>
+  <xacro:arg name="use_nominal_extrinsics" default="true"/>
   <xacro:include filename="$(find patrol_description)/urdf/patrol_wheel.urdf.xacro" />
   <xacro:include filename="$(find sick_scan_xd)/urdf/sick_scan.urdf.xacro" />
@@ -30,5 +30,5 @@
       <origin xyz="0 0 0" rpy="${pi/2} 0 0" />
       <geometry>
-        <mesh filename="package://patrol_description/meshes/ANCS-000-R1.STL" />
+        <mesh filename="package://patrol_description/meshes/ANCS-000-R2.STL" />
       </geometry>
       <material name="white"/>
@@ -43,5 +43,5 @@
   <!-- Drop Z value to ground-->
   <joint name="base_footprint_joint" type="fixed">
-    <origin xyz="0 0 ${wheel_radius}" rpy="0 0 0" />
+    <origin xyz="0 0 ${-wheel_radius}" rpy="0 0 0" />
     <parent link="base_link" />
     <child link="base_footprint" />
@@ -135,11 +135,11 @@
   <xacro:if value="${realsense_enabled}">
     <xacro:sensor_d435i parent="base_link" name="cam0" use_nominal_extrinsics="$(arg use_nominal_extrinsics)">
-      <origin xyz="-0.11913 -0.00228 0.78821" rpy="0 0 0"/>
+      <origin xyz="-0.11913 -0.00228 0.81801" rpy="0 0 0"/>
     </xacro:sensor_d435i>
     <xacro:sensor_d435i parent="base_link" name="cam1" use_nominal_extrinsics="$(arg use_nominal_extrinsics)">
-      <origin xyz="-0.2489 0.1793 0.69821" rpy="0 0 ${pi/2}"/>
+      <origin xyz="-0.2489 0.18991 0.81653" rpy="0 0.122173 ${pi/2}"/>
     </xacro:sensor_d435i>
     <xacro:sensor_d435i parent="base_link" name="cam2" use_nominal_extrinsics="$(arg use_nominal_extrinsics)">
-      <origin xyz="-0.2489 -0.17925 0.69821" rpy="0 0 ${-pi/2}"/>
+      <origin xyz="-0.2489 -0.18991 0.81653" rpy="0 0.122173 ${-pi/2}"/>
     </xacro:sensor_d435i>
   </xacro:if>

Commit message: Changes to base_footprint and base_link frame positions

File: patrol_description/urdf/patrol.urdf.xacro (robot description, xacro)
@@ -43,7 +43,7 @@
   <!-- Drop Z value to ground-->
   <joint name="base_footprint_joint" type="fixed">
-    <origin xyz="0 0 ${-wheel_radius}" rpy="0 0 0" />
-    <parent link="base_link" />
-    <child link="base_footprint" />
+    <origin xyz="0 0 ${wheel_radius}" rpy="0 0 0" />
+    <parent link="base_footprint" />
+    <child link="base_link" />
   </joint>
   <!-- Inertial link stores the robot's inertial information - using husky for timebeing -->
